File: onion2 breakout.sch (KiCad schematic (older format))
At the start: 14 parts, among them P1 USB_B, P2 USB_B, P3 CONN_01X16, P4 CONN_01X16, P5 CONN_01X16, P6 CONN_01X16, U1 CH340G, U2 AP1117, Y1 Crystal

Commit message: Fxed Rx/Tx lines from CH340G to Onion. Adjusted header spacing to accomidate onion. Changed power/data connector from USB B to USB micro. Added BOM.
Parts:
- C1, C2: value C -> 22pF
- C3: value C -> 100uF
- C4: value C -> 10uF
- C5: value C -> 0.1uF
- Y1: value Crystal -> 12MHz
Connections:
- net RxD: now also U1.2 (TXD); no longer U1.3 (RXD)
- net TxD: now also U1.3 (RXD); no longer U1.2 (TXD)
Changed lines of the file:
@@
 P 5150 1250
 F 0 "C3" H 5175 1350 50  0000 L CNN
-F 1 "C" H 5175 1150 50  0000 L CNN
+F 1 "100uF" H 5175 1150 50  0000 L CNN
 F 2 "Capacitors_SMD:C_1206_HandSoldering" H 5188 1100 50  0001 C CNN
 F 3 "" H 5150 1250 50  0000 C CNN
@@
 P 1900 4100
 F 0 "Y1" H 1900 4250 50  0000 C CNN
-F 1 "Crystal" H 1900 3950 50  0000 C CNN
+F 1 "12MHz" H 1900 3950 50  0000 C CNN
 F 2 "Crystals:Crystal_SMD_HC49-SD_HandSoldering" H 1900 4100 50  0001 C CNN
 F 3 "" H 1900 4100 50  0000 C CNN
@@
 P 1400 3950
 F 0 "C1" H 1425 4050 50  0000 L CNN
-F 1 "C" H 1425 3850 50  0000 L CNN
+F 1 "22pF" H 1425 3850 50  0000 L CNN
 F 2 "Capacitors_SMD:C_1206_HandSoldering" H 1438 3800 50  0001 C CNN
 F 3 "" H 1400 3950 50  0000 C CNN
@@
 P 1400 4250
 F 0 "C2" H 1425 4350 50  0000 L CNN
-F 1 "C" H 1425 4150 50  0000 L CNN
+F 1 "22pF" H 1425 4150 50  0000 L CNN
 F 2 "Capacitors_SMD:C_1206_HandSoldering" H 1438 4100 50  0001 C CNN
 F 3 "" H 1400 4250 50  0000 C CNN
@@
 D2-
 Text GLabel 3600 3950 2    60   Input ~ 0
+TxD
+Text GLabel 3600 4050 2    60   Input ~ 0
 RxD
-Text GLabel 3600 4050 2    60   Input ~ 0
-TxD
 Text GLabel 8450 5250 2    60   Input ~ 0
 RxD
@@
 P 6200 1250
 F 0 "C4" H 6225 1350 50  0000 L CNN
-F 1 "C" H 6225 1150 50  0000 L CNN
+F 1 "10uF" H 6225 1150 50  0000 L CNN
 F 2 "Capacitors_SMD:C_1206_HandSoldering" H 6238 1100 50  0001 C CNN
 F 3 "" H 6200 1250 50  0000 C CNN
@@
 P 6450 1250
 F 0 "C5" H 6475 1350 50  0000 L CNN
-F 1 "C" H 6475 1150 50  0000 L CNN
+F 1 "0.1uF" H 6475 1150 50  0000 L CNN
 F 2 "Capacitors_SMD:C_1206_HandSoldering" H 6488 1100 50  0001 C CNN
 F 3 "" H 6450 1250 50  0000 C CNN

Commit message: Corrected issue with u-USB pinout. Moved USB A connector down a bit for more clearance. Rev 2.0
Connections:
- net GND: now also P1.5 (shield); no longer P1.4 (GND)
Other:
- note added: "This is a micro-USB \nconnector. Pin 5 is\nGND and 4 is shield."
Changed lines of the file:
@@
 Title "Onion 2 Breakout"
 Date ""
-Rev ""
+Rev "2"
 Comp ""
 Comment1 ""
@@
 	1    7350 4300
 	-1   0    0    -1
-$EndComp
-$Comp
-L GND #PWR01
-U 1 1 588E1A5D
-P 1300 1500
-F 0 "#PWR01" H 1300 1250 50  0001 C CNN
-F 1 "GND" H 1300 1350 50  0000 C CNN
-F 2 "" H 1300 1500 50  0000 C CNN
-F 3 "" H 1300 1500 50  0000 C CNN
-	1    1300 1500
-	0    -1   -1   0
 $EndComp
 $Comp
@@
 Text GLabel 3600 2300 2    60   Input ~ 0
 D2-
-NoConn ~ 1400 1000
 NoConn ~ 3500 1000
 NoConn ~ 3200 4650
@@
 Wire Wire Line
 	7650 3300 7650 3550
+NoConn ~ 1300 1500
+$Comp
+L GND #PWR?
+U 1 1 58E9570A
+P 1400 1000
+F 0 "#PWR?" H 1400 750 50  0001 C CNN
+F 1 "GND" H 1400 850 50  0000 C CNN
+F 2 "" H 1400 1000 50  0000 C CNN
+F 3 "" H 1400 1000 50  0000 C CNN
+	1    1400 1000
+	0    -1   -1   0
+$EndComp
+Text Notes 650  800  0    60   ~ 0
+This is a micro-USB \nconnector. Pin 5 is\nGND and 4 is shield.
 $EndSCHEMATC
